Commit message: feat(go2): 添加相机传感器支持
在 go2_gazebo.xacro 中添加相机传感器配置：
- camera link: 相机物理链接（小方块可视化）
- camera_joint: 固定关节，安装位置 trunk 前方 (x=0.28m, z=0.05m)
- gazebo camera sensor: 640x480 分辨率，10Hz 帧率，120° 视场角
- 发布话题: /camera/image_raw

影响：RViz Image 模块现在可以显示 go2 相机图像

Closes: RViz Image 模块无图像显示问题

Co-authored-by: Qwen-Coder <qwen-coder@alibabacloud.com>

File: src/gazebo_quadbot/robot_scene/xacro/go2_gazebo.xacro (robot description, xacro)
@@ -187,3 +187,46 @@
         <kd>1.0</kd>
     </gazebo>
+    <!-- Camera link -->
+    <link name="camera">
+        <inertial>
+            <origin xyz="0 0 0" rpy="0 0 0" />
+            <mass value="0.001" />
+            <inertia ixx="0.0001" ixy="0" ixz="0" iyy="0.0001" iyz="0" izz="0.0001" />
+        </inertial>
+        <visual>
+            <origin xyz="0 0 0" rpy="0 0 0" />
+            <geometry>
+                <box size="0.01 0.03 0.01" />
+            </geometry>
+        </visual>
+    </link>
+    <!-- Camera joint -->
+    <joint name="camera_joint" type="fixed">
+        <origin xyz="0.28 0 0.05" rpy="0 0 0" />
+        <parent link="trunk" />
+        <child link="camera" />
+        <axis xyz="0 0 0" />
+    </joint>
+    <!-- Camera sensor -->
+    <gazebo reference="camera">
+        <sensor name="camera" type="camera">
+            <pose>0 0 0 0 0 0</pose>
+            <update_rate>10</update_rate>
+            <camera>
+                <horizontal_fov>2.0944</horizontal_fov>
+                <image>
+                    <width>640</width>
+                    <height>480</height>
+                    <format>R8G8B8</format>
+                </image>
+                <clip>
+                    <near>0.1</near>
+                    <far>100.0</far>
+                </clip>
+            </camera>
+            <plugin name="gazebo_ros_camera" filename="libgazebo_ros_camera.so">
+                <frame_name>camera</frame_name>
+            </plugin>
+        </sensor>
+    </gazebo>
 </robot>
