Commit message: fix(go2w): 降低摩擦系数和关节阻尼以消除足端高频振动
问题原因：
1. 足端摩擦系数 mu1/mu2=3.0 过高（Go2 为 0.6），导致轮子与地面咬合过紧
2. 关节阻尼 damping=0.1 过高（Go2 为 0.01），导致控制器响应过冲

修复内容：
- mu1/mu2: 3.0 → 0.6（与 Go2 一致）
- hip/thigh/calf_damping: 0.1 → 0.01（与 Go2 一致）

影响：消除 Go2W 初始化后足端高频振动和微小移动

Co-authored-by: Qwen-Coder <qwen-coder@alibabacloud.com>

File: src/gazebo_quadbot/robot_scene/xacro/go2w_const.xacro (robot description, xacro)
@@ -60,5 +60,5 @@
     <xacro:property name="hip_velocity_max" value="30.1"/>
     <xacro:property name="hip_torque_max" value="23.7"/>
-    <xacro:property name="hip_damping" value="0.1"/>
+    <xacro:property name="hip_damping" value="0.01"/>
     <xacro:property name="hip_friction" value="0.2"/>
     <xacro:property name="thigh_position_max" value="3.4907"/>
@@ -66,5 +66,5 @@
     <xacro:property name="thigh_velocity_max" value="30.1"/>
     <xacro:property name="thigh_torque_max" value="23.7"/>
-    <xacro:property name="thigh_damping" value="0.1"/>
+    <xacro:property name="thigh_damping" value="0.01"/>
     <xacro:property name="thigh_friction" value="0.2"/>
     <xacro:property name="calf_position_max" value="-0.83776"/>
@@ -72,5 +72,5 @@
     <xacro:property name="calf_velocity_max" value="20.06"/>
     <xacro:property name="calf_torque_max" value="35.55"/>
-    <xacro:property name="calf_damping" value="0.1"/>
+    <xacro:property name="calf_damping" value="0.01"/>
     <xacro:property name="calf_friction" value="0.2"/>
     <xacro:property name="foot_velocity_max" value="30.1"/>

File: src/gazebo_quadbot/robot_scene/xacro/go2w_description.urdf.xacro (robot description, xacro)
@@ -218,6 +218,6 @@
     </joint>
     <gazebo reference="${prefix}_foot">
-        <mu1>3</mu1>
-        <mu2>3</mu2>
+        <mu1>0.6</mu1>
+        <mu2>0.6</mu2>
         <kp>10000.0</kp>
         <kd>1.0</kd>
